File: pcb/_autosave-pcb.sch (KiCad schematic (older format))
At the start: 9 parts, among them J1 Conn_01x02, J2 Conn_01x04_Male, U1 MCP73811T-420I-OT, U2 LD39050PU33R, U3 ESP8266-12E_ESP-12E

Commit message: update the pcb
Parts:
- added U?: BME280, Package_LGA:Bosch_LGA-8_2.5x2.5mm_P0.65mm_ClockwisePinNumbering, symbol Sensor:BME280
Changed lines of the file:
@@
 Wire Wire Line
 	7900 3050 8000 3050
+$Comp
+L Sensor:BME280 U?
+U 1 1 5F0CD6B3
+P 7050 1650
+F 0 "U?" H 6621 1696 50  0000 R CNN
+F 1 "BME280" H 6621 1605 50  0000 R CNN
+F 2 "Package_LGA:Bosch_LGA-8_2.5x2.5mm_P0.65mm_ClockwisePinNumbering" H 8550 1200 50  0001 C CNN
+F 3 "https://ae-bst.resource.bosch.com/media/_tech/media/datasheets/BST-BME280-DS002.pdf" H 7050 1450 50  0001 C CNN
+	1    7050 1650
+	1    0    0    -1
+$EndComp
 $EndSCHEMATC

Commit message: finish the shcematic design
Parts:
- removed D1: D_Schottky, Diode_SMD:D_SMA_Handsoldering, symbol Device:D_Schottky
- removed J2: Conn_01x04_Male, Connector_PinSocket_2.54mm:PinSocket_1x04_P2.54mm_Vertical, symbol Connector:Conn_01x04_Male
- removed RN?: R_Pack04, symbol Device:R_Pack04
- removed U1: MCP73811T-420I-OT, Package_TO_SOT_SMD:SOT-23-5, symbol Battery_Management:MCP73811T-420I-OT
- removed U2: LD39050PU33R, SON95P300X300X100-7N, symbol LD39050PU33R:LD39050PU33R
- removed U3: ESP8266-12E_ESP-12E, XCVR_ESP8266-12E/ESP-12E, symbol ESP8266-12E_ESP-12E:ESP8266-12E_ESP-12E
- removed U?: BME280, Package_LGA:Bosch_LGA-8_2.5x2.5mm_P0.65mm_ClockwisePinNumbering, symbol Sensor:BME280
- added C3: 10u, Capacitor_SMD:C_0603_1608Metric_Pad1.05x0.95mm_HandSolder, symbol Device:C
- added C4: 100nF, Capacitor_SMD:C_0603_1608Metric, symbol Device:C
- added C5, C6, C7: 100n, Capacitor_SMD:C_0603_1608Metric, symbol Device:C
- added D1: SP0503BAHTG, digikey-footprints:SOT-143-4, symbol dk_TVS-Diodes:SP0503BAHTG
- added H1, H2, H3: MountingHole_Pad, MountingHole:MountingHole_3.2mm_M3_DIN965_Pad, symbol Mechanical:MountingHole_Pad
- added H4: MountingHole_Pad, MountingHole:MountingHole_3.2mm_M3, symbol Mechanical:MountingHole_Pad
- added J2: USB_B_Micro, Connector_USB:USB_Micro-B_Molex-105017-0001, symbol Connector:USB_B_Micro
- added Q1: Si2371EDS, Package_TO_SOT_SMD:SOT-23, symbol Transistor_FET:Si2371EDS
- added Q2, Q3: MMBT2222A-TP, digikey-footprints:SOT-23-3, symbol dk_Transistors-Bipolar-BJT-Single:MMBT2222A-TP
- added R1: 2k, Resistor_SMD:R_0603_1608Metric_Pad1.05x0.95mm_HandSolder, symbol Device:R_US
- added R10, R11, R12, R9: 10k, Resistor_SMD:R_0603_1608Metric, symbol Device:R_US
- added R2, R3: 10k, Resistor_SMD:R_0603_1608Metric_Pad1.05x0.95mm_HandSolder, symbol Device:R_US
- added R4: R_Pack04_Split, Resistor_SMD:R_Array_Concave_4x0603, symbol Device:R_Pack04_Split
- added R5, R6: 100k, Resistor_SMD:R_0603_1608Metric_Pad1.05x0.95mm_HandSolder, symbol Device:R_US
- added R7, R8: 10k, Resistor_SMD:R_Array_Concave_4x0603, symbol Device:R_Pack04_Split
- added U1: LD1117S33CTR, digikey-footprints:SOT-223, symbol dk_PMIC-Voltage-Regulators-Linear:LD1117S33CTR
- added U2: MCP73831-2-OT, Package_TO_SOT_SMD:SOT-23-5, symbol Battery_Management:MCP73831-2-OT
- added U3: CP2104, Package_DFN_QFN:QFN-24-1EP_4x4mm_P0.5mm_EP2.6x2.6mm, symbol Interface_USB:CP2104
- added U4: CCS811, Package_LGA:AMS_LGA-10-1EP_2.7x4mm_P0.6mm, symbol Sensor_Gas:CCS811
- added U5: ESP-12F, RF_Module:ESP-12E, symbol RF_Module:ESP-12F
- added U6: BME280, digikey-footprints:Pressure_Sensor_LGA-8_2.5x2.5mm_BME280, symbol dk_Humidity-Moisture-Sensors:BME280
- added U7: TSL2561, Kevin_Lutzer:TSL2561, symbol Kevin_Lutzer:TSL2561
- C1: value 1uf -> 1u
Connections:
- net labels added: BAT_LVL, CCS_nINT, I2C_SCK, I2C_SDA, UART_RX, UART_TX, nBAT_STAT, nBOOT, nINT, nRST
- net labels removed: BOOT, EN, RST, RX, TX
- wire segments 47 -> 163
- no-connect marks 0 -> 26
Other:
- note added: "1K - 1A\n2K - 500mA\n10K - 100mA\n"
- note added: "Lipo Charger and Regulator"
- note added: "Sensor Array"
- note added: "The CP210x series of chips requires a driver. There is also a built in Boot/Rst trigger using the DTR and RTS controls.\nhttps://www.silabs.com/products/development-tools/software/usb-to-uart-bridge-vcp-drivers"
- note added: "USB Bridge"
- moved on the sheet: C1, C2, J1
