File: pcb/_autosave-pcb.kicad_pcb (KiCad board)
At the start: 2 copper layers, 60 x 30 mm, 9 parts, among them J1 USB_B_Mini, SW1 OS102011MA1QN1‎, SW2 PTS645Vx83, SW3 PTS645Vx83, U5 ESP-12F

Commit message: update the pcb stuff
Parts:
- added C1: 100n, Capacitor_SMD:C_0603_1608Metric, F.Cu at (69.5, 42.5)
- added C10: 1u, Capacitor_SMD:C_0603_1608Metric, F.Cu at (69.5, 45.0)
- added C2: 47u, Capacitor_SMD:C_0805_2012Metric, F.Cu at (58.6, 47.2)
- added C3: 100n, Capacitor_SMD:C_0603_1608Metric, F.Cu at (73.5, 45.0)
- added C4: 100n, Capacitor_SMD:C_0603_1608Metric, F.Cu at (131.0, 37.0)
- added C5: 100n, Capacitor_SMD:C_0603_1608Metric, F.Cu at (77.7, 39.1)
- added C6: 100n, Capacitor_SMD:C_0603_1608Metric, F.Cu at (73.7, 39.1)
- added C8: 10u, Capacitor_SMD:C_0805_2012Metric, F.Cu at (73.5, 42.5)
- added C9: 100n, Capacitor_SMD:C_0603_1608Metric, F.Cu at (80.1, 36.6)
- added D1: WS2812B, LED_SMD:LED_WS2812B_PLCC4_5.0x5.0mm_P3.2mm, F.Cu at (60.6, 36.2)
- added D2: SP0503BAHT, Package_TO_SOT_SMD:SOT-143, F.Cu at (67.4, 35.1)
- added J2: Conn_01x04_Male, Connector_PinHeader_2.54mm:PinHeader_1x04_P2.54mm_Vertical, F.Cu at (94.9, 33.4)
- added R2: 10k, Resistor_SMD:R_0603_1608Metric, F.Cu at (76.1, 36.6)
- added R3: 10k, Resistor_SMD:R_0603_1608Metric, F.Cu at (80.1, 34.1)
- added R4: 10k, Resistor_SMD:R_0603_1608Metric, F.Cu at (76.1, 34.1)
- added R5: 10k, Resistor_SMD:R_Array_Convex_4x0603, F.Cu at (64.7, 46.5)
- added RN1: 10k, Resistor_SMD:R_Array_Convex_4x0603, F.Cu at (99.3, 33.5)
- added SW1: PTS645Vx83, Button_Switch_THT:SW_Tactile_SPST_Angled_PTS645Vx58-2LFS, F.Cu at (121.4, 37.5)
- added U1: AP2112K-3.3, Package_TO_SOT_SMD:SOT-23-5, F.Cu at (131.4, 33.4)
- added U2: MIC5225-1.8YM5, Package_TO_SOT_SMD:SOT-23-5, F.Cu at (65.1, 41.8)
- added U3: CP2104, Package_DFN_QFN:QFN-24-1EP_4x4mm_P0.5mm_EP2.6x2.6mm, F.Cu at (59.5, 42.6)
Connections:
- SW1 pad 2: Net-(R2-Pad1) -> (no net)
- U5 pad 14: (no net) -> MODE
