File: pcb/pcb.sch (KiCad schematic (older format))
At the start: 39 parts, among them J1 USB_B_Mini, J4 UART_BUS, Q1 BSS138DW-7-F, SW1 PTS645Vx83, SW2 PTS645Vx83, SW3 PTS645Vx83, SW4 KMR2, U1 AP2112K-3.3, U2 MIC5225-1.8YM5, U3 CP2104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

Commit message: Update the gerbers for the rem v1 and reroute the UART lines
Changed lines of the file:
@@
 NoConn ~ 1750 6700
 NoConn ~ 3000 3150
-Text GLabel 7850 1700 2    50   Output ~ 0
+Text GLabel 7850 1700 2    50   Input ~ 0
 nINT
 $Comp
