File: pcb/pcb.kicad_pcb (KiCad board)
At the start: 2 copper layers, 60 x 30 mm, 54 parts, among them J1 USB_B_Mini, J2 I2C_BUS, J4 UART_BUS, Q1 BSS138DW-7-F, Q2 BSS138DW-7-F, SW1 PTS645Vx83, SW2 PTS645Vx83, SW3 PTS645Vx83, SW4 KMR2, U1 AP2112K-3.3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

Commit message: update the footprint for the tsl2591
Parts:
- turned U7 to 90 degrees
Connections:
- U4 pad 5: (no net) -> GND
- U7 pad 1: +3V3 -> I2C_SCK
- U7 pad 4: I2C_SCK -> (no net)
- U7 pad 5: (no net) -> +3V3
Routing:
- net +3V3: track 18.0 -> 17.0 mm
- net GND: track 48.4 -> 49.3 mm, vias 22 -> 21
- net I2C_SDA: track 40.2 -> 41.0 mm, vias 3 -> 4
Changed lines of the file:
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@@
     (add_net "Net-(U3-Pad24)")
     (add_net "Net-(U3-Pad9)")
-    (add_net "Net-(U4-Pad5)")
     (add_net "Net-(U5-Pad10)")
     (add_net "Net-(U5-Pad11)")
@@
     (add_net "Net-(U5-Pad4)")
     (add_net "Net-(U5-Pad9)")
-    (add_net "Net-(U7-Pad5)")
+    (add_net "Net-(U7-Pad4)")
     (add_net RGB_LED)
     (add_net UART_RX)
@@
   )
   (module Kevin-Lutzer-Kicad-Lbr:TSL2591 (layer F.Cu)
-    (at 69.55 58.6 270)
+    (at 69.55 58.6 90)
     (fp_text reference U7 (at 0.1 2.3 90) (layer F.SilkS)
       (effects (font (size 1 1) (thickness 0.15)))
@@
       (effects (font (size 1 1) (thickness 0.15)))
     )
+    (fp_line (start -1.5 -1.5) (end 1.5 -1.5) (layer F.CrtYd) (width 0.06))
+    (fp_line (start -1.5 1.5) (end -1.5 -1.5) (layer F.CrtYd) (width 0.06))
+    (fp_line (start 1.5 1.5) (end -1.5 1.5) (layer F.CrtYd) (width 0.06))
+    (fp_line (start 1.5 -1.5) (end 1.5 1.5) (layer F.CrtYd) (width 0.06))
+    (fp_line (start 1 1.3) (end 0 1.3) (layer F.SilkS) (width 0.12))
+    (fp_line (start 1 -1.3) (end -1 -1.3) (layer F.SilkS) (width 0.12))
+    (fp_line (start 1 1.2) (end 1 1) (layer F.Fab) (width 0.12))
+    (fp_line (start -1 1.2) (end 1 1.2) (layer F.Fab) (width 0.12))
+    (fp_line (start -1 1) (end -1 1.2) (layer F.Fab) (width 0.12))
+    (fp_line (start -1 -1) (end -1 1) (layer F.Fab) (width 0.12))
+    (fp_line (start -1 -1.2) (end -1 -1) (layer F.Fab) (width 0.12))
+    (fp_line (start 1 -1.2) (end -1 -1.2) (layer F.Fab) (width 0.12))
+    (fp_line (start 1 -1) (end 1 -1.2) (layer F.Fab) (width 0.12))
+    (fp_line (start -1 -1.2) (end 0 -1.2) (layer F.Fab) (width 0.12))
+    (fp_line (start -1 1) (end -1 -1) (layer F.Fab) (width 0.12))
+    (fp_line (start 1 1.2) (end -1 1.2) (layer F.Fab) (width 0.12))
+    (fp_line (start 1 -1) (end 1 1) (layer F.Fab) (width 0.12))
     (fp_line (start 0 -1.2) (end 1 -1.2) (layer F.Fab) (width 0.12))
-    (fp_line (start 1 -1) (end 1 1) (layer F.Fab) (width 0.12))
-    (fp_line (start 1 1.2) (end -1 1.2) (layer F.Fab) (width 0.12))
-    (fp_line (start -1 1) (end -1 -1) (layer F.Fab) (width 0.12))
-    (fp_line (start -1 -1.2) (end 0 -1.2) (layer F.Fab) (width 0.12))
-    (fp_line (start 1 -1) (end 1 -1.2) (layer F.Fab) (width 0.12))
-    (fp_line (start 1 -1.2) (end -1 -1.2) (layer F.Fab) (width 0.12))
-    (fp_line (start -1 -1.2) (end -1 -1) (layer F.Fab) (width 0.12))
-    (fp_line (start -1 -1) (end -1 1) (layer F.Fab) (width 0.12))
-    (fp_line (start -1 1) (end -1 1.2) (layer F.Fab) (width 0.12))
-    (fp_line (start -1 1.2) (end 1 1.2) (layer F.Fab) (width 0.12))
-    (fp_line (start 1 1.2) (end 1 1) (layer F.Fab) (width 0.12))
-    (fp_line (start 1 -1.3) (end -1 -1.3) (layer F.SilkS) (width 0.12))
-    (fp_line (start 1 1.3) (end 0 1.3) (layer F.SilkS) (width 0.12))
-    (fp_line (start 1.5 -1.5) (end 1.5 1.5) (layer F.CrtYd) (width 0.06))
-    (fp_line (start 1.5 1.5) (end -1.5 1.5) (layer F.CrtYd) (width 0.06))
-    (fp_line (start -1.5 1.5) (end -1.5 -1.5) (layer F.CrtYd) (width 0.06))
-    (fp_line (start -1.5 -1.5) (end 1.5 -1.5) (layer F.CrtYd) (width 0.06))
-    (pad 6 smd rect (at 0.75 -0.65 270) (size 1.2 0.35) (layers F.Cu)
+    (pad 6 smd rect (at 0.75 -0.65 90) (size 1.2 0.35) (layers F.Cu F.Paste F.Mask)
       (net 8 I2C_SDA))
-    (pad 5 smd rect (at 0.75 0 270) (size 1.2 0.35) (layers F.Cu))
-    (pad 4 smd rect (at 0.75 0.65 270) (size 1.2 0.35) (layers F.Cu)
+    (pad 5 smd rect (at 0.75 0 90) (size 1.2 0.35) (layers F.Cu F.Paste F.Mask)
+      (net 3 +3V3))
+    (pad 4 smd rect (at 0.75 0.65 90) (size 1.2 0.35) (layers F.Cu F.Paste F.Mask))
+    (pad 3 smd rect (at -0.75 0.65 90) (size 1.2 0.35) (layers F.Cu F.Paste F.Mask)
+      (net 2 GND))
+    (pad 2 smd rect (at -0.75 0 90) (size 1.2 0.35) (layers F.Cu F.Paste F.Mask)
+      (net 19 nINT))
+    (pad 1 smd oval (at -0.75 -0.65 90) (size 1.2 0.35) (layers F.Cu F.Paste F.Mask)
       (net 9 I2C_SCK))
-    (pad 3 smd rect (at -0.75 0.65 270) (size 1.2 0.35) (layers F.Cu)
-      (net 2 GND))
-    (pad 2 smd rect (at -0.75 0 270) (size 1.2 0.35) (layers F.Cu)
-      (net 19 nINT))
-    (pad 1 smd oval (at -0.75 -0.65 270) (size 1.2 0.35) (layers F.Cu)
-      (net 3 +3V3))
   )
   (module Kevin-Lutzer-Kicad-Lbr:SGP30 (layer F.Cu)
@@
       (effects (font (size 0.64 0.64) (thickness 0.015)))
     )
-    (fp_arc (start -0.000005 -0.000005) (end -0.5 -0.225) (angle -318.455) (layer F.Fab) (width 0.2032))
     (fp_poly (pts (xy -0.3 -0.425) (xy 0.3 -0.425) (xy 0.3 0.425) (xy -0.3 0.425)) (layer F.Paste) (width 0.01))
     (fp_circle (center -1.524 -1.524) (end -1.397 -1.524) (layer F.SilkS) (width 0.2032))
@@
     (fp_poly (pts (xy -1.525 -0.2) (xy -0.975 -0.2) (xy -0.975 0.2) (xy -1.525 0.2)) (layer F.Paste) (width 0.01))
     (fp_poly (pts (xy -1.525 -1) (xy -0.975 -1) (xy -0.975 -0.6) (xy -1.525 -0.6)) (layer F.Paste) (width 0.01))
+    (fp_arc (start -0.000005 -0.000005) (end -0.5 -0.225) (angle -318.455) (layer F.Fab) (width 0.2032))
     (pad 5 smd rect (at 1.15 0) (size 0.55 0.4) (layers F.Cu F.Mask)
       (net 11 +1V8))
@@
       (effects (font (size 0.5 0.5) (thickness 0.075)))
     )
-    (pad 5 smd rect (at 0.975 1.025 90) (size 0.5 0.35) (layers F.Cu F.Paste F.Mask))
+    (pad 5 smd rect (at 0.975 1.025 90) (size 0.5 0.35) (layers F.Cu F.Paste F.Mask)
+      (net 2 GND))
     (pad 6 smd rect (at 0.325 1.025 90) (size 0.5 0.35) (layers F.Cu F.Paste F.Mask)
       (net 3 +3V3))
@@
   (segment (start 70.35 64.85) (end 71.15 65.65) (width 0.25) (layer F.Cu) (net 2) (status 10))
   (segment (start 70.2875 64.85) (end 70.35 64.85) (width 0.25) (layer F.Cu) (net 2) (status 30))
-  (via (at 68.075 57.85) (size 0.8) (drill 0.4) (layers F.Cu B.Cu) (net 2))
-  (segment (start 68.9 57.85) (end 68.075 57.85) (width 0.25) (layer F.Cu) (net 2) (status 10))
+  (via (at 68.075 57.85) (size 0.8) (drill 0.4) (layers F.Cu B.Cu) (net 8))
+  (segment (start 68.9 57.85) (end 68.075 57.85) (width 0.25) (layer F.Cu) (net 8) (status 10))
   (via (at 59.75 57.1) (size 0.8) (drill 0.4) (layers F.Cu B.Cu) (net 2))
   (segment (start 59.0375 57.8125) (end 59.75 57.1) (width 0.25) (layer F.Cu) (net 2) (status 10))
@@
   (segment (start 62.75 62.4) (end 64.6 62.4) (width 0.4) (layer F.Cu) (net 2))
   (via (at 64.6 62.4) (size 1.2) (drill 0.6) (layers F.Cu B.Cu) (net 2))
+  (segment (start 70.475 64.5625) (end 70.475 63.075) (width 0.25) (layer F.Cu) (net 2))
+  (segment (start 70.2875 64.75) (end 70.475 64.5625) (width 0.25) (layer F.Cu) (net 2))
   (segment (start 85.0125 75.2) (end 85 75.1875) (width 0.4) (layer F.Cu) (net 3) (status 30))
   (segment (start 87.4 75.2) (end 85.0125 75.2) (width 0.4) (layer F.Cu) (net 3) (status 30))
@@
   (segment (start 68.525 62.714998) (end 68.739999 62.499999) (width 0.25) (layer F.Cu) (net 3))
   (segment (start 68.525 63.075) (end 68.525 62.714998) (width 0.25) (layer F.Cu) (net 3) (status 10))
-  (segment (start 70.2 57.85) (end 70.2 56.825) (width 0.25) (layer F.Cu) (net 3) (status 10))
   (segment (start 74 62.3) (end 74 65.05) (width 0.25) (layer F.Cu) (net 3) (status 10))
   (via (at 66 74.25) (size 0.8) (drill 0.4) (layers F.Cu B.Cu) (net 3))
@@
   (segment (start 72.325001 58.924999) (end 76.223001 58.924999) (width 0.25) (layer B.Cu) (net 9))
   (segment (start 71.025 60.225) (end 72.325001 58.924999) (width 0.25) (layer B.Cu) (net 9))
-  (segment (start 71.025 60.175) (end 70.80001 59.95001) (width 0.25) (layer B.Cu) (net 9))
   (segment (start 71.025 60.225) (end 71.025 60.175) (width 0.25) (layer B.Cu) (net 9))
   (segment (start 75.4 64.7) (end 75.75 65.05) (width 0.25) (layer B.Cu) (net 9))

Commit message: use the right tsl2591 footprint
Parts:
- removed R16: 10k, Resistor_SMD:R_0603_1608Metric
- added D2: LED, LED_SMD:LED_0603_1608Metric, F.Cu at (69.2, 81.4)
- added D5: LED, LED_SMD:LED_0603_1608Metric, F.Cu at (67.2, 81.4)
- added R17: 470, Resistor_SMD:R_0603_1608Metric, F.Cu at (71.2, 78.0)
- added R18: 470, Resistor_SMD:R_0603_1608Metric, F.Cu at (69.2, 78.0)
- added R19: 470, Resistor_SMD:R_0603_1608Metric, F.Cu at (67.2, 78.0)
- D1: value WS2812B -> LED; footprint LED_SMD:LED_WS2812B_PLCC4_5.0x5.0mm_P3.2mm -> LED_SMD:LED_0603_1608Metric
- U4: footprint Package_LGA:Bosch_LGA-8_2.5x2.5mm_P0.65mm_ClockwisePinNumbering -> digikey-footprints:Pressure_Sensor_LGA-8_2.5x2.5mm_BME280
- moved D1 4.95 mm to (71.2, 81.4), turned to 90 degrees
- turned U7 to 270 degrees
Connections:
- D1 pad 1: +3V3 -> GND
- D1 pad 2: (no net) -> Net-(D1-Pad2)
- U4 pad 2: Net-(R16-Pad2) -> +3V3
- U5 pad 10: (no net) -> SIG2
- U5 pad 11: (no net) -> SIG1
- U5 pad 19: I2C_SCK -> I2C_SDA
- U5 pad 20: I2C_SDA -> I2C_SCK
- U5 pad 6: RGB_LED -> (no net)
- U5 pad 9: (no net) -> SIG3
Routing:
- net RGB_LED: track 15.3 -> 0.00 mm, vias 2 -> 0
- net SIG1: track 0.00 -> 9.51 mm
- net SIG2: track 0.00 -> 7.15 mm
- net GND: track 49.3 -> 54.0 mm, vias 21 -> 22
- net SIG3: track 0.00 -> 3.85 mm
- net Net-(R16-Pad2): track 3.63 -> 0.00 mm
- net I2C_SCK: track 43.6 -> 40.6 mm
- net Net-(D5-Pad2): track 0.00 -> 1.79 mm
- net Net-(D2-Pad2): track 0.00 -> 1.79 mm
- net Net-(D1-Pad2): track 0.00 -> 1.79 mm
- net I2C_SDA: track 41.0 -> 40.2 mm, vias 4 -> 3

Commit message: cleaning up logic
Connections:
- R12 pad 2: I2C_SDA -> I2C_SCK
- R13 pad 2: I2C_SCK -> I2C_SDA
Routing:
- net I2C_SCK: track 40.6 -> 45.2 mm
- net I2C_SDA: track 40.2 -> 37.6 mm
- net +3V3: track 17.0 -> 14.8 mm
- net GND: track 54.0 -> 55.4 mm
- net I2C_SCK_1V8: track 10.2 -> 10.9 mm
Other:
- board text added: "Room Environment Monitor Kevin Luzer Rev B"
- board text removed: "Room Environment Monitor Kevin Luzer Rev A"
