File: pcb/sensors.sch (KiCad schematic (older format))
At the start: 12 parts, among them J2 I2C_BUS, Q2 BSS138DW-7-F, U4 BME280, U6 SGP30

Commit message: WIP
Parts:
- gave numbers to parts that had none: 1
Changed lines of the file:
@@
 Connection ~ 2150 2000
 $Comp
-L Kevin_Lutzer:TSL2591 U?
+L Kevin_Lutzer:TSL2591 U7
 U 1 1 5FFE72E4
 P 3850 1350
-F 0 "U?" H 3550 1650 50  0000 L CNN
+F 0 "U7" H 3550 1650 50  0000 L CNN
 F 1 "TSL2591" H 3850 1650 50  0000 L CNN
 F 2 "Kevin-Lutzer-Kicad-Lbr:TSL2591" H 3300 1100 50  0001 C CNN

Commit message: cleaning up logic
Connections:
- net I2C_SCK: now also R12.2; no longer R13.2
- net I2C_SDA: now also R13.2; no longer R12.2
Other:
- moved on the sheet: C12, R10, R11, R12, R13, U6
Changed lines of the file:
@@
 I2C_SDA
 Wire Wire Line
-	1550 5450 1550 5500
-Wire Wire Line
-	1550 5500 1650 5500
-Wire Wire Line
-	1750 5500 1750 5450
-Wire Wire Line
-	1650 5450 1650 5500
-Connection ~ 1650 5500
-Wire Wire Line
-	1650 5500 1750 5500
+	1550 5600 1550 5650
+Wire Wire Line
+	1550 5650 1650 5650
+Wire Wire Line
+	1750 5650 1750 5600
+Wire Wire Line
+	1650 5600 1650 5650
+Connection ~ 1650 5650
+Wire Wire Line
+	1650 5650 1750 5650
 $Comp
 L power:GND #PWR?
 U 1 1 5F9ABC5B
-P 1650 5500
+P 1650 5650
 AR Path="/5F9ABC5B" Ref="#PWR?"  Part="1"
 AR Path="/5F9A85F1/5F9ABC5B" Ref="#PWR0118"  Part="1"
-F 0 "#PWR0118" H 1650 5250 50  0001 C CNN
-F 1 "GND" H 1655 5327 50  0000 C CNN
-F 2 "" H 1650 5500 50  0001 C CNN
-F 3 "" H 1650 5500 50  0001 C CNN
-	1    1650 5500
+F 0 "#PWR0118" H 1650 5400 50  0001 C CNN
+F 1 "GND" H 1655 5477 50  0000 C CNN
+F 2 "" H 1650 5650 50  0001 C CNN
+F 3 "" H 1650 5650 50  0001 C CNN
+	1    1650 5650
 	1    0    0    -1
 $EndComp
 Wire Wire Line
 	1150 3400 1400 3400
-$Comp
-L power:+1V8 #PWR?
-U 1 1 5F9ABC63
-P 1650 4800
-AR Path="/5F9ABC63" Ref="#PWR?"  Part="1"
-AR Path="/5F9A85F1/5F9ABC63" Ref="#PWR0119"  Part="1"
-F 0 "#PWR0119" H 1650 4650 50  0001 C CNN
-F 1 "+1V8" H 1665 4973 50  0000 C CNN
-F 2 "" H 1650 4800 50  0001 C CNN
-F 3 "" H 1650 4800 50  0001 C CNN
-	1    1650 4800
-	1    0    0    -1
-$EndComp
-Wire Wire Line
-	1650 4800 1600 4800
-Wire Wire Line
-	1600 4800 1600 4850
-Wire Wire Line
-	1700 4850 1700 4800
-Wire Wire Line
-	1700 4800 1650 4800
-Connection ~ 1650 4800
 $Comp
 L power:+1V8 #PWR?
 U 1 1 5F9ABC6E
-P 2100 4650
+P 2100 4700
 AR Path="/5F9ABC6E" Ref="#PWR?"  Part="1"
 AR Path="/5F9A85F1/5F9ABC6E" Ref="#PWR0120"  Part="1"
-F 0 "#PWR0120" H 2100 4500 50  0001 C CNN
-F 1 "+1V8" H 2115 4823 50  0000 C CNN
-F 2 "" H 2100 4650 50  0001 C CNN
-F 3 "" H 2100 4650 50  0001 C CNN
-	1    2100 4650
-	1    0    0    -1
-$EndComp
-Wire Wire Line
-	2250 5100 2100 5100
-Wire Wire Line
-	2100 4700 2100 4650
+F 0 "#PWR0120" H 2100 4550 50  0001 C CNN
+F 1 "+1V8" H 2115 4873 50  0000 C CNN
+F 2 "" H 2100 4700 50  0001 C CNN
+F 3 "" H 2100 4700 50  0001 C CNN
+	1    2100 4700
+	1    0    0    -1
+$EndComp
+Wire Wire Line
+	2150 5250 2100 5250
+Wire Wire Line
+	2100 4850 2100 4700
 $Comp
 L power:+1V8 #PWR?
 U 1 1 5F9ABC79
-P 1150 4650
+P 1150 4700
 AR Path="/5F9ABC79" Ref="#PWR?"  Part="1"
 AR Path="/5F9A85F1/5F9ABC79" Ref="#PWR0121"  Part="1"
-F 0 "#PWR0121" H 1150 4500 50  0001 C CNN
-F 1 "+1V8" H 1165 4823 50  0000 C CNN
-F 2 "" H 1150 4650 50  0001 C CNN
-F 3 "" H 1150 4650 50  0001 C CNN
-	1    1150 4650
-	1    0    0    -1
-$EndComp
-Wire Wire Line
-	1150 4700 1150 4650
-Wire Wire Line
-	1050 5100 1150 5100
+F 0 "#PWR0121" H 1150 4550 50  0001 C CNN
+F 1 "+1V8" H 1165 4873 50  0000 C CNN
+F 2 "" H 1150 4700 50  0001 C CNN
+F 3 "" H 1150 4700 50  0001 C CNN
+	1    1150 4700
+	1    0    0    -1
+$EndComp
+Wire Wire Line
+	1150 4850 1150 4700
+Wire Wire Line
+	1050 5250 1150 5250
 $Comp
 L power:+3.3V #PWR?
@@
 Wire Wire Line
 	4250 4550 4400 4550
-Text GLabel 1050 5100 0    50   Input ~ 0
+Text GLabel 1050 5250 0    50   Input ~ 0
 I2C_SDA_1V8
-Text GLabel 2250 5100 2    50   Input ~ 0
+Text GLabel 2150 5250 2    50   Input ~ 0
 I2C_SCK_1V8
 Text GLabel 2050 4000 2    50   Output ~ 0
@@
 	1900 3700 2000 3700
 Wire Wire Line
-	2100 5000 2100 5100
-Connection ~ 2100 5100
-Wire Wire Line
-	2100 5100 2050 5100
-Wire Wire Line
-	1150 5000 1150 5100
-Connection ~ 1150 5100
-Wire Wire Line
-	1150 5100 1250 5100
+	2100 5150 2100 5250
+Connection ~ 2100 5250
+Wire Wire Line
+	2100 5250 2050 5250
+Wire Wire Line
+	1150 5150 1150 5250
+Connection ~ 1150 5250
+Wire Wire Line
+	1150 5250 1250 5250
 $Comp
 L Connector:Conn_01x04_Male J2
@@
 L Device:C C12
 U 1 1 5F40EB79
-P 3050 5100
-F 0 "C12" H 3165 5146 50  0000 L CNN
-F 1 "100n" H 3165 5055 50  0000 L CNN
-F 2 "Capacitor_SMD:C_0603_1608Metric" H 3088 4950 50  0001 C CNN
-F 3 "~" H 3050 5100 50  0001 C CNN
-	1    3050 5100
+P 2950 5000
+F 0 "C12" H 3065 5046 50  0000 L CNN
+F 1 "100n" H 3065 4955 50  0000 L CNN
+F 2 "Capacitor_SMD:C_0603_1608Metric" H 2988 4850 50  0001 C CNN
+F 3 "~" H 2950 5000 50  0001 C CNN
+	1    2950 5000
 	1    0    0    -1
 $EndComp
@@
 L power:GND #PWR0142
 U 1 1 5F40F86F
-P 3050 5300
-F 0 "#PWR0142" H 3050 5050 50  0001 C CNN
-F 1 "GND" H 3055 5127 50  0000 C CNN
-F 2 "" H 3050 5300 50  0001 C CNN
-F 3 "" H 3050 5300 50  0001 C CNN
-	1    3050 5300
+P 2950 5200
+F 0 "#PWR0142" H 2950 4950 50  0001 C CNN
+F 1 "GND" H 2955 5027 50  0000 C CNN
+F 2 "" H 2950 5200 50  0001 C CNN
+F 3 "" H 2950 5200 50  0001 C CNN
+	1    2950 5200
 	1    0    0    -1
 $EndComp
@@
 	1    0    0    -1
 $EndComp
-$Comp
-L power:+1V8 #PWR0144
-U 1 1 5F41045C
-P 3050 4900
-F 0 "#PWR0144" H 3050 4750 50  0001 C CNN
-F 1 "+1V8" H 3065 5073 50  0000 C CNN
-F 2 "" H 3050 4900 50  0001 C CNN
-F 3 "" H 3050 4900 50  0001 C CNN
-	1    3050 4900
-	1    0    0    -1
-$EndComp
-Wire Wire Line
-	3050 4950 3050 4900
 Wire Wire Line
 	4300 1700 4300 1650
@@
 	4300 2000 4300 2050
 Wire Wire Line
-	3050 5250 3050 5300
+	2950 5150 2950 5200
 Wire Wire Line
 	1300 3200 1300 3700
@@
 L Device:R_US R10
 U 1 1 5F42F459
-P 1150 4850
-F 0 "R10" H 1218 4896 50  0000 L CNN
-F 1 "10k" H 1218 4805 50  0000 L CNN
-F 2 "Resistor_SMD:R_0603_1608Metric" V 1190 4840 50  0001 C CNN
-F 3 "~" H 1150 4850 50  0001 C CNN
-	1    1150 4850
+P 1150 5000
+F 0 "R10" H 1218 5046 50  0000 L CNN
+F 1 "10k" H 1218 4955 50  0000 L CNN
+F 2 "Resistor_SMD:R_0603_1608Metric" V 1190 4990 50  0001 C CNN
+F 3 "~" H 1150 5000 50  0001 C CNN
+	1    1150 5000
 	1    0    0    -1
 $EndComp
@@
 L Device:R_US R11
 U 1 1 5F431D99
-P 2100 4850
-F 0 "R11" H 2168 4896 50  0000 L CNN
-F 1 "10k" H 2168 4805 50  0000 L CNN
-F 2 "Resistor_SMD:R_0603_1608Metric" V 2140 4840 50  0001 C CNN
-F 3 "~" H 2100 4850 50  0001 C CNN
-	1    2100 4850
+P 2100 5000
+F 0 "R11" H 2168 5046 50  0000 L CNN
+F 1 "10k" H 2168 4955 50  0000 L CNN
+F 2 "Resistor_SMD:R_0603_1608Metric" V 2140 4990 50  0001 C CNN
+F 3 "~" H 2100 5000 50  0001 C CNN
+	1    2100 5000
 	1    0    0    -1
 $EndComp
@@
 L Device:R_US R12
 U 1 1 5F43299F
+P 4400 4800
+F 0 "R12" H 4468 4846 50  0000 L CNN
+F 1 "10k" H 4468 4755 50  0000 L CNN
+F 2 "Resistor_SMD:R_0603_1608Metric" V 4440 4790 50  0001 C CNN
+F 3 "~" H 4400 4800 50  0001 C CNN
+	1    4400 4800
+	1    0    0    -1
+$EndComp
+$Comp
+L Device:R_US R13
+U 1 1 5F437086
 P 4050 4800
-F 0 "R12" H 4118 4846 50  0000 L CNN
+F 0 "R13" H 4118 4846 50  0000 L CNN
 F 1 "10k" H 4118 4755 50  0000 L CNN
 F 2 "Resistor_SMD:R_0603_1608Metric" V 4090 4790 50  0001 C CNN
@@
 	1    0    0    -1
 $EndComp
-$Comp
-L Device:R_US R13
-U 1 1 5F437086
-P 4400 4800
-F 0 "R13" H 4468 4846 50  0000 L CNN
-F 1 "10k" H 4468 4755 50  0000 L CNN
-F 2 "Resistor_SMD:R_0603_1608Metric" V 4440 4790 50  0001 C CNN
-F 3 "~" H 4400 4800 50  0001 C CNN
-	1    4400 4800
-	1    0    0    -1
-$EndComp
 Wire Wire Line
 	4400 4950 4400 5250
@@
 L Kevin_Lutzer:SGP30 U6
 U 1 1 5F5E68DD
-P 1650 5150
-F 0 "U6" H 1850 5400 50  0000 L CNN
-F 1 "SGP30" H 1800 4900 50  0000 L CNN
-F 2 "Kevin-Lutzer-Kicad-Lbr:SGP30" H 1600 5850 50  0001 C CNN
-F 3 "" H 1650 5100 50  0001 C CNN
-	1    1650 5150
+P 1650 5300
+F 0 "U6" H 1850 5550 50  0000 L CNN
+F 1 "SGP30" H 1800 5050 50  0000 L CNN
+F 2 "Kevin-Lutzer-Kicad-Lbr:SGP30" H 1600 6000 50  0001 C CNN
+F 3 "" H 1650 5250 50  0001 C CNN
+	1    1650 5300
 	1    0    0    -1
 $EndComp
@@
 	1    0    0    -1
 $EndComp
+$Comp
+L power:+1V8 #PWR?
+U 1 1 5FFBD6B0
+P 1700 4700
+AR Path="/5FFBD6B0" Ref="#PWR?"  Part="1"
+AR Path="/5F9A85F1/5FFBD6B0" Ref="#PWR0119"  Part="1"
+F 0 "#PWR0119" H 1700 4550 50  0001 C CNN
+F 1 "+1V8" H 1715 4873 50  0000 C CNN
+F 2 "" H 1700 4700 50  0001 C CNN
+F 3 "" H 1700 4700 50  0001 C CNN
+	1    1700 4700
+	1    0    0    -1
+$EndComp
+Wire Wire Line
+	1700 4700 1700 4950
+Wire Wire Line
+	1600 4950 1700 4950
+Wire Wire Line
+	1600 4950 1600 5000
+Connection ~ 1700 4950
+Wire Wire Line
+	1700 4950 1700 5000
+$Comp
+L power:+1V8 #PWR?
+U 1 1 600722B4
+P 2950 4700
+AR Path="/600722B4" Ref="#PWR?"  Part="1"
+AR Path="/5F9A85F1/600722B4" Ref="#PWR?"  Part="1"
+F 0 "#PWR?" H 2950 4550 50  0001 C CNN
+F 1 "+1V8" H 2965 4873 50  0000 C CNN
+F 2 "" H 2950 4700 50  0001 C CNN
+F 3 "" H 2950 4700 50  0001 C CNN
+	1    2950 4700
+	1    0    0    -1
+$EndComp
+Wire Wire Line
+	2950 4700 2950 4850
 $EndSCHEMATC
