File: pcb/sensors.kicad_sch (KiCad schematic)
At the start: 22 parts, among them J2 Conn_01x04_Pin, Q1 BSS138, Q2 BSS138, U3 BME280, U4 SGP30-2.5K

Commit message: add the routing for hte PM1006K enable, and other fixes
Connections:
- net GND: now also D6.2 (A); no longer D6.1 (K)
- net PD: now also D6.1 (K); no longer D6.2 (A)
- net PM1006_GND: now reaches J2.4 (Pin_4), JP1.2 (B), Q2.3 (D)
Other:
- moved on the sheet: D6
Changed lines of the file:
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@@
+    (effects (font (size 1.27 1.27)) (justify left bottom))
+  )
+  (label "PM1006_GND" (at 101.6 143.51 0) (fields_autoplaced)
     (effects (font (size 1.27 1.27)) (justify left bottom))
   )
@@
     )
   )
-  (symbol (lib_id "Device:D_Photo") (at 102.87 102.87 90) (unit 1)
-    (in_bom yes) (on_board yes) (dnp no) (fields_autoplaced)
-    (property "Reference" "D6" (at 94.615 103.8225 0)
-      (effects (font (size 1.27 1.27)))
-    )
-    (property "Value" "D_Photo" (at 97.155 103.8225 0)
-      (effects (font (size 1.27 1.27)))
+  (symbol (lib_id "Device:D_Photo") (at 102.87 105.41 270) (unit 1)
+    (in_bom yes) (on_board yes) (dnp no) (fields_autoplaced)
+    (property "Reference" "D6" (at 107.95 103.1875 90)
+      (effects (font (size 1.27 1.27)) (justify left))
+    )
+    (property "Value" "D_Photo" (at 107.95 105.7275 90)
+      (effects (font (size 1.27 1.27)) (justify left))
     )
     (property "Footprint" "Diode_SMD:D_1206_3216Metric_Pad1.42x1.75mm_HandSolder" (at 102.87 104.14 0)
