File: pcb/sensors.kicad_sch (KiCad schematic)
At the start: 20 parts, among them J2 Conn_01x04_Pin, Q1 BSS138, U3 BME280, U4 SGP30-2.5K

Commit message: Kevinlutzer/upgrade to v8 (#11)
* Add new plugins for BOM and PNP file management

* make some more progress

* merge in main

* cleanup sensors

* pass drc

* move files

* rename files

* lint and add justfile

* add the just file

* add github actions

* WIP

* platformio build

* redo the build command

* od this in the right directory

* update workflow

* use local libs

* lint

* lint

* ignore format

* build

* lint

* install clang format

* cleanup

* rename firmware files

* add vscode and platformio updates

* finish off firmware.ini

* delete uneeded pipelines

* update lint command ran

* use the firmware name

* firmware again
Parts:
- removed U4: SGP30-2.5K, Kevin_Lutzer_Lbr:SGP30-2.5K_SEN, symbol Kevin_Lutzer_Lbr:SGP30-2.5K
- added TP5, TP6: TestPoint, TestPoint:TestPoint_Pad_D1.0mm, symbol Connector:TestPoint
- added U3: SGP40, Kevin_Lutzer_Lbr:SGP30-2.5K_SEN-M, symbol Kevin_Lutzer_Lbr:SGP40
- C2, C4: renamed from C8; DNP (none) -> C1590
- C5: DNP (none) -> C1590
- C7: renamed from C6; DNP (none) -> C1592
- D6: now not fitted; now left out of the parts list
- J2: DNP (none) -> C265083
- Q1: DNP (none) -> C52895
- R10, R11: renamed from R5; DNP (none) -> C4190
- R12, R13, R3: renamed from R5; DNP (none) -> C15401
- R14: value R_Small_US -> 10M; now not fitted; now left out of the parts list
- R4: renamed from R5; DNP (none) -> C23164
- R8, R9: renamed from R5; DNP (none) -> C15402
- TP2: renamed from TP3; now not fitted; now left out of the parts list
- TP3: renamed from TP2; now not fitted; now left out of the parts list
- U4: renamed from U3; DNP (none) -> C92489
Connections:
- net +3V3: now also U3.5 (VDDH); no longer U4.2 (CSB)
- net GND: now also U4.2 (CSB), U3.2 (VSS), U3.4 (N/A), U3.7 (PAD)
- net I2C_SCL: now also TP6.1, U3.6 (SCL)
- net I2C_SDA: now also TP5.1, U3.3 (SDA)
- net SGP30_VDD: now also U3.1 (VDD)
Other:
- moved on the sheet: C2, C4, C5, C7, J2, R10, R12, R13, R3, R4, R8, R9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
