File: pcb/room_environment_monitor.kicad_sch (KiCad schematic)
At the start: 37 parts, among them J1 Conn_01x02_Pin, J3 Conn_01x06_Socket, P1 USB_C_Plug_USB2.0, Q2 BSS138, Q3 BSS138, U1 ESP32-C3-WROOM-02, U5 AP2112K-3.3

Commit message: finish layout for factory reset
Parts:
- added SW1: SW_SPST, Button_Switch_SMD:SW_Push_1P1T_NO_CK_KMR2, symbol Switch:SW_SPST
- D3, D4, D5: value SK6812MINI -> WS2812B-2020; symbol LED:SK6812MINI -> LED:WS2812B-2020; DPN (none) -> C965555; now fitted; now in the parts list
- P1: now fitted; now in the parts list
- U1: DNP (none) -> C2934560
Connections:
- net GND: now also SW1.1 (A)
- net FACT_REST: now reaches U1.17 (GPIO1/ADC1_CH1/XTAL_32K_N)
- net FACT_REST: now also SW1.2 (B)
- no-connect marks 8 -> 7
Other:
- note added: "Factory Reset"
- note added: "Uses internal pullup"
- moved on the sheet: C3, C6
